File: SolarRegulator-pcba/SolarRegulator.kicad_pcb (KiCad board)
At the start: 2 copper layers, 78 parts, among them J2 Screw_Terminal_01x02, J3 1x03, J5 1x02, Q1 DMP2165UW, Q2 DMN2004WKQ, Q3 DMP2165UW, U1 TPS63802DLAR, U2 SPV1040T, U3 L6924D

Commit message: Add final footprints, update LED footprints to 1206
Parts:
- added C15: 100nF, Capacitor_SMD:C_0805_2012Metric_Pad1.15x1.40mm_HandSolder, F.Cu at (205.4, 71.4)
- added C7: 1uF, Capacitor_SMD:C_1206_3216Metric_Pad1.42x1.75mm_HandSolder, F.Cu at (206.0, 68.3)
- added D7: SMM4F5.0A-TR, SMM4FxxA:SMM4FxxA, F.Cu at (203.8, 65.9)
- added J1: USB_B_Micro, Connector_USB:USB_Micro-B_Molex-105017-0001, F.Cu at (167.8, 64.7)
- added J4: Conn_01x05, Connector_PinHeader_2.54mm:PinHeader_1x05_P2.54mm_Vertical, F.Cu at (160.6, 64.1)
- added JP1: 4.2(o=4.1V), Jumper:SolderJumper-2_P1.3mm_Bridged_RoundedPad1.0x1.5mm, F.Cu at (210.0, 71.7)
- added L1: 10uH, MSS7341-103ML:MSS7341-103ML, F.Cu at (163.1, 47.4)
- D1, D2, D3, D4, D5, D6: footprint LED_THT:LED_D5.0mm -> LED_SMD:LED_1206_3216Metric
- Q2: footprint Package_TO_SOT_SMD:SOT-323_SC-70 -> Package_TO_SOT_SMD:SOT-323_SC-70_Handsoldering
- moved C1 274.5 mm to (53.2, 30.8)
- moved C10 274.5 mm to (70.5, 33.9)
- moved C11 274.5 mm to (69.6, 37.2)
- moved C13 274.5 mm to (64.5, 43.1)
- moved C14 274.5 mm to (69.3, 40.2)
- moved C2 274.5 mm to (69.3, 43.1)
- moved C3 274.5 mm to (47.3, 36.8)
- moved C4 274.5 mm to (63.3, 46.1)
- moved C8 274.5 mm to (64.5, 40.2)
- moved C9 274.5 mm to (58.6, 43.8)
- moved L2 274.5 mm to (39.1, 31.1)
- moved R10 274.5 mm to (41.3, 40.1)
- moved R11 274.5 mm to (41.3, 33.5)
- moved R12 274.5 mm to (66.4, 27.5)
- moved R15 274.5 mm to (53.2, 37.4)
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Connections:
- BT1 pad 1: /Power/VBATT_IN -> +BATT
- C2 pad 1: /Power/VBATT_IN -> +BATT
- C4 pad 1: /Power/VBATT_IN -> +BATT
- TP7 pad 1: /Power/VBATT_IN -> +BATT
- U1 pad 1: /Power/VBATT_IN -> +BATT
- U1 pad 10: /Power/VBATT_IN -> +BATT
